File: projects/four-switch-insert/circuits/circuits.kicad_pcb (KiCad board)
At the start: 2 copper layers, 45 x 45 mm, 33 parts, among them J1 Screw_Terminal_01x02, J3 Screw_Terminal_01x02, Q1 BT136-500, SW1 SW_Push, SW2 SW_Push, SW3 SW_Push, SW4 SW_Push, U1 ESP-WROOM-02, U2 MOC3033M

Commit message: a lot of changes
Parts:
- added J2: AC MAINS CONN, TerminalBlock:TerminalBlock_bornier-3_P5.08mm, B.Cu at (116.2, 31.0)
- J1: value Screw_Terminal_01x02 -> BACK_PCB; footprint TerminalBlock_WAGO_Local:TerminalBlock_WAGO_2061_1x02_P6.00mm -> Connector_PinHeader_2.54mm:PinHeader_1x03_P2.54mm_Vertical
- J3: value Screw_Terminal_01x02 -> FRONT_PCB; footprint TerminalBlock_WAGO_Local:TerminalBlock_WAGO_2061_1x02_P6.00mm -> Connector_PinHeader_2.54mm:PinHeader_1x03_P2.54mm_Vertical; moved to F.Cu
- PS1: value IRM-02-3.3S -> HLK-PM03; footprint Converter_ACDC:Converter_ACDC_MeanWell_IRM-02-xx_SMD -> Converter_ACDC:Converter_ACDC_HiLink_HLK-PMxx; moved to F.Cu
- Q1: footprint Package_TO_SOT_THT:TO-220-3_Vertical -> Package_TO_SOT_SMD:TO-252-2
- R9: moved to B.Cu
- U2: footprint Package_DIP:DIP-4_W7.62mm_SMDSocket_SmallPads -> Package_DIP:DIP-6_W7.62mm_LongPads
- moved U2 95.9 mm to (88.0, 41.8), turned to 0 degrees
- moved R9 88.2 mm to (85.2, 41.9)
- moved R11 69.6 mm to (110.2, 44.0)
- moved PS1 65.9 mm to (114.5, 41.5)
- moved Q1 55.6 mm to (106.2, 39.2)
- moved J3 46.7 mm to (59.5, 67.5), turned to 180 degrees
- moved D5 27.9 mm to (58.4, 43.9)
- moved R10 27.9 mm to (58.4, 39.4), turned to 90 degrees
- moved C1 22.6 mm to (57.0, 35.0), turned to 90 degrees
- moved U1 15.1 mm to (47.0, 41.0)
- moved 3v3 14.7 mm to (43.2, 69.8)
- moved J1 11.7 mm to (88.8, 48.8), turned to 270 degrees
- moved TP2 10.2 mm to (53.3, 69.8)
- moved R1 10.0 mm to (35.0, 33.5)
- moved TP4 7.47 mm to (45.7, 69.8)
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- renumbered TP1 to 3v3, TP5 to GND
Connections:
- J3 pad 1: Net-(J1-Pad1) -> /AC_PWR_SIG
- J3 pad 2: Net-(J3-Pad2) -> +3V3
- PS1 pad 1: Net-(J1-Pad1) -> Net-(J2-Pad2)
- PS1 pad 3: (no net) -> Net-(J1-Pad1)
- Q1 pad 1: Net-(J1-Pad1) -> Net-(J2-Pad2)
- Q1 pad 2: Net-(J1-Pad2) -> Net-(J2-Pad3)
- R9 pad 2: /AC_PWR_SIG -> Net-(J1-Pad3)
- U2 pad 2: GND -> Net-(J1-Pad1)
Other:
- board size 45 x 45 mm -> 91.4 x 42.8 mm
