File: projects/four-switch-insert/circuits/circuits.sch (KiCad schematic (older format))
At the start: 33 parts, among them J1 Screw_Terminal_01x02, J3 Screw_Terminal_01x02, Q1 BT136-500, SW1 SW_Push, SW2 SW_Push, SW3 SW_Push, SW4 SW_Push, U1 ESP-WROOM-02, U2 MOC3033M

Commit message: a lot of changes
Parts:
- removed J1, J3: Screw_Terminal_01x02, TerminalBlock_WAGO_Local:TerminalBlock_WAGO_2061_1x02_P6.00mm, symbol Connector:Screw_Terminal_01x02
- removed PS1: IRM-02-3.3S, Converter_ACDC:Converter_ACDC_MeanWell_IRM-02-xx_SMD, symbol Converter_ACDC:IRM-02-3.3S
- added J1: BACK_PCB, Connector_PinHeader_2.54mm:PinHeader_1x03_P2.54mm_Vertical, symbol Connector:Conn_01x03_Male
- added J2: AC MAINS CONN, TerminalBlock:TerminalBlock_bornier-3_P5.08mm, symbol Connector:Screw_Terminal_01x03
- added J3: FRONT_PCB, Connector_PinHeader_2.54mm:PinHeader_1x03_P2.54mm_Vertical, symbol Connector:Conn_01x03_Male
- added PS1: HLK-PM03, Converter_ACDC:Converter_ACDC_HiLink_HLK-PMxx, symbol Converter_ACDC:HLK-PM03
- Q1: footprint Package_TO_SOT_THT:TO-220-3_Vertical -> Package_TO_SOT_SMD:TO-252-2
- U2: footprint Package_DIP:DIP-4_W7.62mm_SMDSocket_SmallPads -> Package_DIP:DIP-6_W7.62mm_LongPads
Connections:
- wire segments 91 -> 100
Other:
- moved on the sheet: C2, C3, C4, C5, R1, R2, R3, R4, R5, R6, R7, R8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
