File: lkf-series/circuits/front-pcb/front-pcb.kicad_pcb (KiCad board)
At the start: 2 copper layers, 41.3 x 41.5 mm, 21 parts, among them J1 Inter_PCB_Conn, SW1 SW_Push, SW2 SW_Push, SW3 SW_Push, SW4 SW_Push, U1 ESP-12F

Commit message: lkf series pcbs traced and mostly ready for order
Parts:
- added J7: Prog_Conn, Connector_PinSocket_2.54mm:PinSocket_2x03_P2.54mm_Vertical, B.Cu at (86.5, 40.0)
- added LED1: WS2812C-2020_SW1, WS2812C-2020:WS2812C2020, F.Cu at (87.3, 25.6)
- added LED2: WS2812C-2020_SW2, WS2812C-2020:WS2812C2020, F.Cu at (69.3, 25.6)
- added LED3: WS2812C-2020_SW3, WS2812C-2020:WS2812C2020, F.Cu at (60.3, 52.6)
- added LED4: WS2812C-2020_SW4, WS2812C-2020:WS2812C2020, F.Cu at (96.3, 52.6)
- moved C2 6.98 mm to (84.0, 31.9), turned to 180 degrees
- moved C3 6.85 mm to (72.5, 31.9), turned to 0 degrees
- moved C4 3.57 mm to (72.5, 57.6), turned to 0 degrees
- moved R7 3.39 mm to (84.0, 30.1), turned to 0 degrees
- moved R8 3.35 mm to (72.5, 30.1), turned to 180 degrees
- moved R5 2.82 mm to (72.4, 61.4), turned to 180 degrees
- moved C5 2.68 mm to (84.1, 54.0)
- moved R10 1.20 mm to (84.1, 55.8)
- moved R2 1.03 mm to (72.5, 55.7)
- moved R1 1.00 mm to (72.5, 53.9)
- moved R6 0.97 mm to (84.1, 57.7)
- moved R4 0.63 mm to (72.5, 28.3), turned to 180 degrees
- moved R3 0.53 mm to (84.0, 28.3), turned to 0 degrees
- moved C1 0.27 mm to (88.0, 54.0)
- moved R9 0.07 mm to (72.5, 59.5), turned to 180 degrees
Connections:
- net Net-(R1-Pad1) renamed /RST
- J1 pad 2: /AC_PWR_CTL -> /AC_PWR_CTRL
- U1 pad 11: /SW3 -> Net-(U1-Pad11)
- U1 pad 12: /SW4 -> Net-(U1-Pad12)
- U1 pad 16: Net-(U1-Pad16) -> /SW1
- U1 pad 17: Net-(U1-Pad17) -> /LED_CTRL
- U1 pad 18: Net-(U1-Pad18) -> /GPIO0
- U1 pad 19: /AC_PWR_CTL -> Net-(U1-Pad19)
- U1 pad 20: /SW1 -> /SW2
- U1 pad 21: Net-(U1-Pad21) -> /RXD
- U1 pad 22: Net-(U1-Pad22) -> /TXD
- U1 pad 4: Net-(U1-Pad4) -> /SW3
- U1 pad 5: /SW2 -> /AC_PWR_CTRL
- U1 pad 6: Net-(U1-Pad6) -> /SW4
Routing:
- net +3V3: track 0.00 -> 179.1 mm, vias 0 -> 1
- net Net-(LED3-Pad1): track 0.00 -> 37.0 mm, vias 0 -> 2
- net Net-(LED2-Pad1): track 0.00 -> 34.7 mm, vias 0 -> 2
- net /RST: track 0.00 -> 20.8 mm
- net Net-(LED1-Pad1): track 0.00 -> 19.0 mm, vias 0 -> 2
- net /SW3: track 0.00 -> 16.8 mm
- net /SW2: track 0.00 -> 16.5 mm
- net /LED_CTRL: track 0.00 -> 13.4 mm, vias 0 -> 2
- net /TXD: track 0.00 -> 12.5 mm
- net Net-(R5-Pad2): track 0.00 -> 11.7 mm
- net /AC_PWR_CTRL: track 0.00 -> 10.9 mm
- net Net-(R3-Pad2): track 0.00 -> 10.8 mm
- net Net-(R6-Pad2): track 0.00 -> 10.8 mm
- net Net-(R4-Pad2): track 0.00 -> 10.8 mm
- net /SW1: track 0.00 -> 9.44 mm
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- added copper zone on B.Cu, net GND
- added copper zone on F.Cu, net GND
Other:
- board text added: "3v3"
- board text added: "GND"
- board text added: "GPIO0"
- board text added: "RST"
- board text added: "RXD"
- board text added: "TXD"
