File: lkf-series/circuits/front-pcb/front-pcb.sch (KiCad schematic (older format))
At the start: 21 parts, among them J1 Inter_PCB_Conn, SW1 SW_Push, SW2 SW_Push, SW3 SW_Push, SW4 SW_Push, U1 ESP-12F

Commit message: lkf series pcbs traced and mostly ready for order
Parts:
- added J7: Prog_Conn, Connector_PinSocket_2.54mm:PinSocket_2x03_P2.54mm_Vertical, symbol Connector_Generic:Conn_01x06
- added LED1: WS2812C-2020_SW1, WS2812C-2020:WS2812C2020, symbol WS2812C-2020:WS2812C-2020
- added LED2: WS2812C-2020_SW2, WS2812C-2020:WS2812C2020, symbol WS2812C-2020:WS2812C-2020
- added LED3: WS2812C-2020_SW3, WS2812C-2020:WS2812C2020, symbol WS2812C-2020:WS2812C-2020
- added LED4: WS2812C-2020_SW4, WS2812C-2020:WS2812C2020, symbol WS2812C-2020:WS2812C-2020
Connections:
- net +3V3: now also J7.2 (Pin_2), LED1.4 (VDD), LED2.4 (VDD), LED3.4 (VDD), LED4.4 (VDD)
- net GND: now also J7.1 (Pin_1), LED1.2 (GND), LED2.2 (GND), LED3.2 (GND), LED4.2 (GND)
- net SW1: now also U1.16 (GPIO15); no longer U1.20 (GPIO5)
- net SW2: now also U1.20 (GPIO5); no longer U1.5 (GPIO14)
- net SW3: now also U1.4 (GPIO16); no longer U1.11 (GPIO9)
- net SW4: now also U1.6 (GPIO12); no longer U1.12 (GPIO10)
- net RST: now reaches R1.1, U1.1 (~RST)
- net RST: now also J7.4 (Pin_4)
- net LED_CTRL: now reaches U1.17 (GPIO2)
- net LED_CTRL: now also LED1.3 (DI)
- net GPIO0: now reaches U1.18 (GPIO0)
- net GPIO0: now also J7.3 (Pin_3)
- net RXD: now reaches U1.21 (GPIO3/RXD)
- net RXD: now also J7.5 (Pin_5)
- net TXD: now reaches U1.22 (GPIO1/TXD)
- net TXD: now also J7.6 (Pin_6)
- net AC_PWR_CTL: no longer names the net of U1.19 (GPIO4)
- net AC_PWR_CTL: no longer J1.2 (Pin_2)
- new net: LED1.1 (DO), LED2.3 (DI)
- new net: LED2.1 (DO), LED3.3 (DI)
- new net: LED3.1 (DO), LED4.3 (DI)
- new net AC_PWR_CTRL: J1.2 (Pin_2), U1.5 (GPIO14)
- no-connect marks 13 -> 10
Other:
- moved on the sheet: C1, C2, C3, C4, C5, J1, R1, R10, R2, R3, R4, R5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
