File: roller-shades/circuits/driver-board/driver-board.sch (KiCad schematic (older format))
At the start: 39 parts, among them J1 1B_Conn, J2 DS18B20, J3 Connector_Board_Conn, J4 PROG, J5 WINDOW, J6 1A_Conn, J7 2A_Conn, J8 2B_Conn, U1 AMS1117-3.3, U2 AS5601-ASOM, U3 DRV5033A1, U4 ESP-12F

Commit message: Refractored dependencies into each project and added missing folders
Parts:
- removed A1: Pololu_Breakout_A4988, Module:Pololu_Breakout-16_15.2x20.3mm, symbol Driver_Motor:Pololu_Breakout_A4988
- removed C1: 100µF, Capacitor_SMD:CP_Elec_6.3x7.7, symbol Device:CP_Small
- removed C3, C6: 10µF, Capacitor_SMD:C_0603_1608Metric, symbol Device:CP_Small
- removed C4, C5: 100nF, Capacitor_SMD:C_0603_1608Metric, symbol Device:CP_Small
- removed D1: DIODE, Diode_SMD:D_0805_2012Metric, symbol Simulation_SPICE:DIODE
- removed F1: Fuse, Fuse:Fuse_0603_1608Metric, symbol Device:Fuse
- removed J1: 1B_Conn, TestPoint:TestPoint_Pad_2.5x2.5mm, symbol Connector_Generic:Conn_01x01
- removed J3: Connector_Board_Conn, Connector_PinHeader_2.00mm:PinHeader_1x06_P2.00mm_Vertical, symbol Connector_Generic:Conn_01x06
- removed J4: PROG, Connector_PinHeader_2.00mm:PinHeader_1x06_P2.00mm_Vertical, symbol Connector_Generic:Conn_01x06
- removed J5: WINDOW, Connector_PinHeader_2.54mm:PinHeader_1x02_P2.54mm_Vertical, symbol Connector_Generic:Conn_01x02
- removed J6: 1A_Conn, TestPoint:TestPoint_Pad_2.5x2.5mm, symbol Connector_Generic:Conn_01x01
- removed J7: 2A_Conn, TestPoint:TestPoint_Pad_2.5x2.5mm, symbol Connector_Generic:Conn_01x01
- removed J8: 2B_Conn, TestPoint:TestPoint_Pad_2.5x2.5mm, symbol Connector_Generic:Conn_01x01
- removed R10, R11, R12, R13, R14, R15, R16, R8, R9: 10k, Resistor_SMD:R_0603_1608Metric, symbol Device:R_Small
- removed U1: AMS1117-3.3, Package_TO_SOT_SMD:SOT-223-3_TabPin2, symbol Regulator_Linear:AMS1117-3.3
- removed U3: DRV5033A1, Package_TO_SOT_THT:TO-92Flat, symbol Sensor_Magnetic:DRV5033AJQDBZ
- removed U4: ESP-12F, RF_Module:ESP-12E, symbol RF_Module:ESP-12F
- added C1: 10µF 50V, Capacitor_SMD:C_0805_2012Metric, symbol Device:C_Small
- added C3: 100nF, Capacitor_SMD:C_0805_2012Metric, symbol Device:C_Small
- added C4: 220pF, Capacitor_SMD:C_0805_2012Metric, symbol Device:C_Small
- added C5: NS, Capacitor_SMD:C_0805_2012Metric, symbol Device:C_Small
- added C6: 22µF 6.3V, Capacitor_SMD:C_0805_2012Metric, symbol Device:C_Small
- added D1: D_Small, symbol Device:D_Small
- added J1: PWR_IN (5-20V), symbol Connector:Screw_Terminal_01x02
- added J3: AUX2, Connector_PinSocket_2.00mm:PinSocket_1x03_P2.00mm_Vertical, symbol Connector_Generic:Conn_01x03
- added J4: Conn_01x04, symbol Connector_Generic:Conn_01x04
- added J5: Conn_01x06, symbol Connector_Generic:Conn_01x06
- added L1: 10uH, symbol Device:L_Small
- added U1: ESP32-WROOM-32, RF_Module:ESP32-WROOM-32, symbol RF_Module:ESP32-WROOM-32
- added U5: MP1584, symbol SHP_Deps:MP1584
- C2, C7: footprint Capacitor_SMD:C_0603_1608Metric -> Capacitor_SMD:C_0805_2012Metric
- C8: value 100nF -> 100µF; footprint Fuse:Fuse_0805_2012Metric -> Capacitor_SMD:C_0805_2012Metric
- J2: value DS18B20 -> AUX1
- R1: value 10k -> 100K; footprint Resistor_SMD:R_0603_1608Metric -> Resistor_SMD:R_0805_2012Metric; LCSC C365360 -> (none)
- R2: value 10k -> 24.9K; footprint Resistor_SMD:R_0603_1608Metric -> Resistor_SMD:R_0805_2012Metric; LCSC C365360 -> (none)
- R3: value 10k -> 200K; footprint Resistor_SMD:R_0603_1608Metric -> Resistor_SMD:R_0805_2012Metric; LCSC C365360 -> (none)
- R4: value 10k -> 68.1K; footprint Resistor_SMD:R_0603_1608Metric -> Resistor_SMD:R_0805_2012Metric; LCSC C365360 -> (none)
- R5: value 220k -> 124K; footprint Resistor_SMD:R_0603_1608Metric -> Resistor_SMD:R_0805_2012Metric; LCSC C365360 -> (none)
- R6: value 100k -> 40.2K; footprint Resistor_SMD:R_0603_1608Metric -> Resistor_SMD:R_0805_2012Metric; LCSC C365360 -> (none)
- R7: value 1K -> 10K; footprint Resistor_SMD:R_0603_1608Metric -> Resistor_SMD:R_0805_2012Metric; LCSC C365360 -> (none)
Connections:
- net labels added: AS5601_ABI_A, AS5601_ABI_B, CONN_AUX1, CONN_AUX2, TMC2209_DIAG, TMC2209_DIR, TMC2209_EN, TMC2209_PDN, TMC2209_RX, TMC2209_STEP, TMC2209_TX, VBUS
- net labels removed: ENC_A, ENC_B, GPIO0, GPIO12, GPIO16, GPIO2, GPIO_ADC, RST, RXD, STEPPER_1A, STEPPER_1B, STEPPER_2A, STEPPER_2B, STPR_DIR, STPR_ENA, STPR_MS1, STPR_MS2, STPR_MS3, STPR_STP, TXD, VDD
- wire segments 152 -> 106
- no-connect marks 7 -> 1
Other:
- moved on the sheet: C2, J2, U2
