File: roller-shades/circuits/driver-board-dev/driver-board.sch (KiCad schematic (older format))
At the start: 22 parts, among them J1 NEMA17_Conn, J2 DS18B20_Conn, J3 Power_Conn, J4 Window_Conn, J5 A3144_Conn, U1 AMS1117-5.0, U2 AS5601-ASOM, U4 WeMos_D1_mini

Commit message: Refractored dependencies into each project and added missing folders
Parts:
- removed A1: Pololu_Breakout_A4988, Module:Pololu_Breakout-16_15.2x20.3mm, symbol Driver_Motor:Pololu_Breakout_A4988
- removed C3, C6: 10µF, Capacitor_SMD:C_0603_1608Metric, symbol Device:CP_Small
- removed C4, C7: 100nF, Capacitor_SMD:C_0603_1608Metric, symbol Device:CP_Small
- removed D1: DIODE, Diode_SMD:D_0805_2012Metric, symbol Simulation_SPICE:DIODE
- removed J1: NEMA17_Conn, Connector_PinHeader_2.54mm:PinHeader_1x04_P2.54mm_Horizontal, symbol Connector_Generic:Conn_01x04
- removed J3: Power_Conn, Connector_PinHeader_2.54mm:PinHeader_1x02_P2.54mm_Vertical, symbol Connector_Generic:Conn_01x02
- removed J4: Window_Conn, Connector_PinHeader_2.54mm:PinHeader_1x03_P2.54mm_Vertical, symbol Connector_Generic:Conn_01x03
- removed J5: A3144_Conn, Package_TO_SOT_THT:TO-92Flat, symbol Connector_Generic:Conn_01x03
- removed U1: AMS1117-5.0, Package_TO_SOT_SMD:SOT-223-3_TabPin2, symbol Regulator_Linear:AMS1117-5.0
- removed U4: WeMos_D1_mini, Module:WEMOS_D1_mini_light, symbol MCU_Module:WeMos_D1_mini
- added A1: BigTreeTech_TMC2209_V12, SHP_Deps:BigTreeTech_TMC22xx_Breakout-16_15.2x20.3mm, symbol SHP_Deps:BigTreeTech_TMC2209_V12
- added C8: 100µF, Capacitor_THT:CP_Radial_D5.0mm_P2.50mm, symbol Device:CP_Small
- added H1, H2, H3, H4: MountingHole, MountingHole:MountingHole_3.2mm_M3_DIN965_Pad, symbol Mechanical:MountingHole
- added J3, J4: Conn_01x01_Female, TestPoint:TestPoint_THTPad_4.0x4.0mm_Drill2.0mm, symbol Connector:Conn_01x01_Female
- added R6: 10K, Resistor_SMD:R_0805_2012Metric_Pad1.20x1.40mm_HandSolder, symbol Device:R_Small
- added U1: DM0x-DC-DC, SHP_Deps:DM02-DC-DC, symbol SHP_Deps:DM0x-DC-DC
- added U3: mini_esp32, SHP_Deps:Wemos_D1_mini32, symbol SHP_Deps:mini_esp32
- added U4: DS18S20, Package_TO_SOT_THT:TO-92_Inline, symbol Sensor_Temperature:DS18S20
- C1: value 100µF -> 100nF; footprint Capacitor_THT:CP_Radial_D8.0mm_P3.50mm -> Capacitor_SMD:C_0805_2012Metric
- C2: footprint Capacitor_SMD:C_0603_1608Metric -> Capacitor_SMD:C_0805_2012Metric
- J2: value DS18B20_Conn -> AUX1
- R1, R2: value 10k -> 10K; footprint Resistor_SMD:R_0603_1608Metric -> Resistor_SMD:R_0805_2012Metric_Pad1.20x1.40mm_HandSolder; LCSC C365360 -> (none)
- R3, R4, R5: value 10k -> 1k; footprint Resistor_SMD:R_0603_1608Metric -> Resistor_SMD:R_0805_2012Metric_Pad1.20x1.40mm_HandSolder; LCSC C365360 -> (none)
- R7: value 1K -> 10K; footprint Resistor_SMD:R_0603_1608Metric -> Resistor_SMD:R_0805_2012Metric_Pad1.20x1.40mm_HandSolder; LCSC C365360 -> (none)
Connections:
- net labels added: AS5601_ABI_A, AS5601_ABI_B, CONN_AUX1, CONN_AUX2, I2C_SCL, I2C_SDA, TEMP_SENSOR, TMC2209_DIAG, TMC2209_DIR, TMC2209_EN, TMC2209_PDN, TMC2209_STEP, VBUS
- net labels removed: +5V, ENC_A, ENC_B, GPIO12, ROLLER_SIG, STPR_DIR, STPR_ENA, STPR_MS1, STPR_MS2, STPR_MS3, STPR_STP, VDD, WINDOW_SIG
- wire segments 102 -> 95
- no-connect marks 8 -> 12
Other:
- moved on the sheet: C2, J2, U2
